File: board/maxm8q_board/maxm8q_board.kicad_pcb (KiCad board)
At the start: 2 copper layers, 46 x 46 mm, 37 parts, among them CN1 AFC12-S02CCC-00, J1 microusb, J2 Conn_02x04_Odd_Even, J4 Conn_02x04_Odd_Even, Q1 BC817, Q2 AO3401A, U1 MAX-M8Q, U2 TPS71730, U3 BL8573CB6TR, X1 ANTENNA_SMA

Commit message: sma
Parts:
- X1: footprint Connector_Coaxial:SMA_Amphenol_132289_EdgeMount -> Connector_Coaxial:SMA_Samtec_SMA-J-P-X-ST-EM1_EdgeMount
- moved X1 0.32 mm to (143.4, 83.1), turned to 90 degrees
- renumbered RESET to SW1
