File: board/maxm8q_board/maxm8q_board.sch (KiCad schematic (older format))
At the start: 37 parts, among them CN1 AFC12-S02CCC-00, J1 microusb, J2 Conn_02x04_Odd_Even, J4 Conn_02x04_Odd_Even, Q1 BC817, Q2 AO3401A, SW1 SW_Push, U1 MAX-M8Q, U2 TPS71730, U3 BL8573CB6TR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

Commit message: sma
Parts:
- X1: footprint Connector_Coaxial:SMA_Amphenol_132289_EdgeMount -> Connector_Coaxial:SMA_Samtec_SMA-J-P-X-ST-EM1_EdgeMount
Changed lines of the file:
@@
 F 0 "X1" H 7550 3000 42  0000 C CNN
 F 1 "ANTENNA_SMA" H 7750 2750 42  0000 C CNN
-F 2 "Connector_Coaxial:SMA_Amphenol_132289_EdgeMount" H 7650 2850 50  0001 C CNN
+F 2 "Connector_Coaxial:SMA_Samtec_SMA-J-P-X-ST-EM1_EdgeMount" H 7650 2850 50  0001 C CNN
 F 3 "" H 7650 2850 50  0001 C CNN
 	1    7650 2850
